File: input_stage.kicad_sch (KiCad schematic)
At the start: 5 parts, among them U2 TL074

Commit message: added LCSC part numbers
Parts:
- R4: LCSC (none) -> C2930232
- R5: LCSC (none) -> C2907295
- R6: LCSC (none) -> C26115
Changed lines of the file:
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@@
+      (effects (font (size 1.27 1.27)) hide)
+    )
+    (property "LCSC" "C26115" (at 100.33 110.49 0)
       (effects (font (size 1.27 1.27)) hide)
     )
@@
     )
     (property "Datasheet" "~" (at 118.11 100.33 0)
+      (effects (font (size 1.27 1.27)) hide)
+    )
+    (property "LCSC" "C2907295" (at 118.11 100.33 0)
       (effects (font (size 1.27 1.27)) hide)
     )
@@
       (effects (font (size 1.27 1.27)) hide)
     )
+    (property "LCSC" "C2930232" (at 149.86 110.49 0)
+      (effects (font (size 1.27 1.27)) hide)
+    )

Commit message: added schema pdf
Other:
- title: (none) -> EQD Plume Clone
Changed lines of the file:
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@@
 (kicad_sch (version 20230121) (generator eeschema)
   (paper "A4")
+  (title_block
+    (title "EQD Plume Clone")
+    (date "2023-08-31")
+    (rev "A")
+  )
   (junction (at 100.33 100.33) (diameter 0) (color 0 0 0 0)
   )
