File: output_stage.kicad_sch (KiCad schematic)
At the start: 9 parts, among them U2 TL074

Commit message: added LCSC part numbers
Parts:
- C11: LCSC (none) -> C32635
- R14: LCSC (none) -> C2907295
- R15: LCSC (none) -> C26115
- R16: LCSC (none) -> C2907294
- R17: LCSC (none) -> C2907293
Changed lines of the file:
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@@
+      (effects (font (size 1.27 1.27)) hide)
+    )
+    (property "LCSC" "~" (at 111.76 93.345 0)
       (effects (font (size 1.27 1.27)) hide)
     )
@@
       (effects (font (size 1.27 1.27)) hide)
     )
+    (property "LCSC" "C2907295" (at 82.55 86.36 0)
+      (effects (font (size 1.27 1.27)) hide)
+    )
     (pin "1")
     (pin "2")
@@
     )
     (property "Datasheet" "~" (at 194.945 90.805 0)
+      (effects (font (size 1.27 1.27)) hide)
+    )
+    (property "LCSC" "C2907294" (at 194.945 90.805 0)
       (effects (font (size 1.27 1.27)) hide)
     )
@@
     )
     (property "Datasheet" "~" (at 203.2 97.79 0)
+      (effects (font (size 1.27 1.27)) hide)
+    )
+    (property "LCSC" "C2907293" (at 203.2 97.79 0)
       (effects (font (size 1.27 1.27)) hide)
     )
@@
       (effects (font (size 1.27 1.27)) hide)
     )
-    (property "LCSC" "" (at 180.34 90.805 0)
+    (property "LCSC" "C32635" (at 180.34 90.805 0)
       (effects (font (size 1.27 1.27)) hide)
     )
@@
       (effects (font (size 1.27 1.27)) hide)
     )
+    (property "LCSC" "C26115" (at 144.145 104.775 0)
+      (effects (font (size 1.27 1.27)) hide)
+    )

Commit message: added schema pdf
Other:
- title: (none) -> EQD Plume Clone
Changed lines of the file:
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@@
 (kicad_sch (version 20230121) (generator eeschema)
   (paper "A4")
+  (title_block
+    (title "EQD Plume Clone")
+    (date "2023-08-31")
+    (rev "A")
+  )
   (junction (at 144.145 93.345) (diameter 0) (color 0 0 0 0)
   )
