File: plumeclone.kicad_sch (KiCad schematic)
At the start: 2 parts, among them J2 FromGuitar_conn_01x02, J3 ToAmplifier_conn_01x02

Commit message: added schema pdf
Other:
- title: (none) -> EQD Plume Clone
Changed lines of the file:
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@@
 (kicad_sch (version 20230121) (generator eeschema)
   (paper "A4")
+  (title_block
+    (title "EQD Plume Clone")
+    (date "2023-08-31")
+    (rev "A")
+  )
   (wire (pts (xy 43.18 123.19) (xy 49.53 123.19))
     (stroke (width 0) (type default))
