File: power_supply.kicad_sch (KiCad schematic)
At the start: 9 parts, among them U2 TL074, U3 TC7660SEOA713

Commit message: added LCSC part numbers
Parts:
- C12, C13: LCSC (none) -> C32635
- D1, D8: footprint (none) -> LED_SMD:LED_0805_2012Metric_Pad1.15x1.40mm_HandSolder; LCSC (none) -> C965812
- R19, R20: LCSC (none) -> C2907305
Changed lines of the file:
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@@
       (effects (font (size 1.27 1.27)) hide)
     )
-    (property "LCSC" "" (at 158.115 116.84 0)
+    (property "LCSC" "C32635" (at 158.115 116.84 0)
       (effects (font (size 1.27 1.27)) hide)
     )
@@
       (effects (font (size 1.27 1.27)) hide)
     )
+    (property "LCSC" "C2907305" (at 207.01 74.93 0)
+      (effects (font (size 1.27 1.27)) hide)
+    )
     (pin "1")
     (pin "2")
@@
       (effects (font (size 1.27 1.27)) (justify left))
     )
-    (property "Footprint" "" (at 206.375 115.57 0)
+    (property "Footprint" "LED_SMD:LED_0805_2012Metric_Pad1.15x1.40mm_HandSolder" (at 206.375 115.57 0)
       (effects (font (size 1.27 1.27)) hide)
     )
     (property "Datasheet" "~" (at 206.375 115.57 0)
+      (effects (font (size 1.27 1.27)) hide)
+    )
+    (property "LCSC" "C965812" (at 206.375 115.57 0)
       (effects (font (size 1.27 1.27)) hide)
     )
@@
       (effects (font (size 1.27 1.27)) hide)
     )
-    (property "LCSC" "" (at 136.525 92.71 0)
+    (property "LCSC" "C32635" (at 136.525 92.71 0)
       (effects (font (size 1.27 1.27)) hide)
     )
@@
     )
     (property "Datasheet" "~" (at 102.235 76.2 0)
+      (effects (font (size 1.27 1.27)) hide)
+    )
+    (property "LCSC" "~" (at 102.235 76.2 0)
       (effects (font (size 1.27 1.27)) hide)
     )
@@
       (effects (font (size 1.27 1.27)) hide)
     )
+    (property "LCSC" "C2907305" (at 206.375 106.68 0)
+      (effects (font (size 1.27 1.27)) hide)
+    )
     (pin "1")
     (pin "2")
@@
       (effects (font (size 1.27 1.27)) (justify right))
     )
-    (property "Footprint" "" (at 207.01 83.82 0)
+    (property "Footprint" "LED_SMD:LED_0805_2012Metric_Pad1.15x1.40mm_HandSolder" (at 207.01 83.82 0)
       (effects (font (size 1.27 1.27)) hide)
     )
@@
       (effects (font (size 1.27 1.27)) hide)
     )
+    (property "LCSC" "C965812" (at 207.01 83.82 0)
+      (effects (font (size 1.27 1.27)) hide)
+    )

Commit message: added schema pdf
Other:
- title: (none) -> EQD Plume Clone
Changed lines of the file:
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@@
 (kicad_sch (version 20230121) (generator eeschema)
   (paper "A4")
+  (title_block
+    (title "EQD Plume Clone")
+    (date "2023-08-31")
+    (rev "A")
+  )
   (junction (at 116.205 69.85) (diameter 0) (color 0 0 0 0)
   )
