File: tone_stage.kicad_sch (KiCad schematic)
At the start: 9 parts, among them U2 TL074

Commit message: added LCSC part numbers
Parts:
- C6: LCSC (none) -> C476766
- C7: LCSC (none) -> C282770
- C8: LCSC (none) -> C106843
- R10, R12: LCSC (none) -> C2907295
- R11: LCSC (none) -> C2930231
- R13: LCSC (none) -> C2930157
Changed lines of the file:
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@@
       (effects (font (size 1.27 1.27)) hide)
     )
-    (property "LCSC" "" (at 135.255 50.165 0)
+    (property "LCSC" "C106843" (at 135.255 50.165 0)
       (effects (font (size 1.27 1.27)) hide)
     )
@@
     )
     (property "Datasheet" "~" (at 173.99 64.77 0)
+      (effects (font (size 1.27 1.27)) hide)
+    )
+    (property "LCSC" "C2907295" (at 173.99 64.77 0)
       (effects (font (size 1.27 1.27)) hide)
     )
@@
       (effects (font (size 1.27 1.27)) hide)
     )
+    (property "LCSC" "~" (at 135.255 64.77 0)
+      (effects (font (size 1.27 1.27)) hide)
+    )
     (pin "1")
     (pin "2")
@@
       (effects (font (size 1.27 1.27)) hide)
     )
-    (property "LCSC" "" (at 125.095 114.3 0)
+    (property "LCSC" "C476766" (at 125.095 114.3 0)
       (effects (font (size 1.27 1.27)) hide)
     )
@@
       (effects (font (size 1.27 1.27)) hide)
     )
+    (property "LCSC" "C2907295" (at 94.615 106.68 0)
+      (effects (font (size 1.27 1.27)) hide)
+    )
     (pin "1")
     (pin "2")
@@
       (effects (font (size 1.27 1.27)) hide)
     )
+    (property "LCSC" "C2930157" (at 116.205 43.18 0)
+      (effects (font (size 1.27 1.27)) hide)
+    )
     (pin "1")
     (pin "2")
@@
       (effects (font (size 1.27 1.27)) hide)
     )
+    (property "LCSC" "C2930231" (at 148.59 114.3 0)
+      (effects (font (size 1.27 1.27)) hide)
+    )
     (pin "1")
     (pin "2")
@@
       (effects (font (size 1.27 1.27)) hide)
     )
-    (property "LCSC" "" (at 173.99 77.47 0)
-      (effects (font (size 1.27 1.27)) hide)
-    )
+    (property "LCSC" "C282770" (at 173.99 77.47 0)
+      (effects (font (size 1.27 1.27)) hide)
+    )

Commit message: added schema pdf
Other:
- title: (none) -> EQD Plume Clone
Changed lines of the file:
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@@
 (kicad_sch (version 20230121) (generator eeschema)
   (paper "A4")
+  (title_block
+    (title "EQD Plume Clone")
+    (date "2023-08-31")
+    (rev "A")
+  )
   (junction (at 160.02 77.47) (diameter 0) (color 0 0 0 0)
   )
